File: MDC64Padapter.kicad_sch (KiCad schematic)
At the start: 36 parts, among them J1 DB9_F_TO_C64, J2 DB9_M_TO_PAD, Q1 BC847, Q2 BC847, SW1 MODE, U1 74ACT08, U2 74ACT373, U3 74ACT157, U4 74ACT373, U5 74AHC1G04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

Commit message: Fix 555 cap/resistor values
Parts:
- C1: value 10uF -> 10nF
- R7: value 47K -> 10K
Changed lines of the file:
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@@
 	(label "MD_UP"
 		(at 248.92 41.91 0)
-		(fields_autoplaced yes)
 		(effects
 			(font
@@
 	(label "C64_POTY"
 		(at 21.59 63.5 90)
-		(fields_autoplaced yes)
 		(effects
 			(font
@@
 	(label "MD_DOWN"
 		(at 233.68 35.56 180)
-		(fields_autoplaced yes)
 		(effects
 			(font
@@
 	(label "C64_B"
 		(at 81.28 30.48 270)
-		(fields_autoplaced yes)
 		(effects
 			(font
@@
 	(label "C64_B"
 		(at 128.27 92.71 180)
-		(fields_autoplaced yes)
 		(effects
 			(font
@@
 	(label "C64_RIGHT"
 		(at 195.58 25.4 180)
-		(fields_autoplaced yes)
 		(effects
 			(font
@@
 	(label "MD_LEFT_M"
 		(at 248.92 31.75 0)
-		(fields_autoplaced yes)
 		(effects
 			(font
@@
 	(label "MD_C{slash}~{ST}"
 		(at 248.92 24.13 0)
-		(fields_autoplaced yes)
 		(effects
 			(font
@@
 	(label "MD_B"
 		(at 95.25 151.13 180)
-		(fields_autoplaced yes)
 		(effects
 			(font
@@
 	(label "C64_B"
 		(at 144.78 38.1 180)
-		(fields_autoplaced yes)
 		(effects
 			(font
@@
 	(label "MD_C{slash}~{ST}"
 		(at 30.48 148.59 0)
-		(fields_autoplaced yes)
 		(effects
 			(font
@@
 	(label "MD_START"
 		(at 180.34 148.59 180)
-		(fields_autoplaced yes)
 		(effects
 			(font
@@
 	(label "CLK"
 		(at 248.92 34.29 0)
-		(fields_autoplaced yes)
 		(effects
 			(font
@@
 	(label "MD_C{slash}~{ST}"
 		(at 115.57 148.59 0)
-		(fields_autoplaced yes)
 		(effects
 			(font
@@
 	(label "MD_START"
 		(at 72.39 87.63 0)
-		(fields_autoplaced yes)
 		(effects
 			(font
@@
 	(label "MD_START"
 		(at 19.05 90.17 0)
-		(fields_autoplaced yes)
 		(effects
 			(font
@@
 	(label "MD_A"
 		(at 19.05 85.09 0)
-		(fields_autoplaced yes)
 		(effects
 			(font
@@
 	(label "C64_DOWN"
 		(at 195.58 35.56 180)
-		(fields_autoplaced yes)
 		(effects
 			(font
@@
 	(label "MD_B"
 		(at 233.68 38.1 180)
-		(fields_autoplaced yes)
 		(effects
 			(font
@@
 	(label "CLK"
 		(at 35.56 171.45 0)
-		(fields_autoplaced yes)
 		(effects
 			(font
@@
 	(label "MD_C"
 		(at 72.39 92.71 0)
-		(fields_autoplaced yes)
 		(effects
 			(font
@@
 	(label "~{CLK}"
 		(at 199.39 109.22 0)
-		(fields_autoplaced yes)
 		(effects
 			(font
@@
 	(label "MD_A"
 		(at 180.34 151.13 180)
-		(fields_autoplaced yes)
 		(effects
 			(font
@@
 	(label "C64_UP"
 		(at 128.27 77.47 180)
-		(fields_autoplaced yes)
 		(effects
 			(font
@@
 	(label "MD_LEFT"
 		(at 95.25 153.67 180)
-		(fields_autoplaced yes)
 		(effects
 			(font
@@
 	(label "~{CLK}"
 		(at 120.65 171.45 0)
-		(fields_autoplaced yes)
 		(effects
 			(font
@@
 	(label "MD_B{slash}~{A}"
 		(at 30.48 151.13 0)
-		(fields_autoplaced yes)
 		(effects
 			(font
@@
 	(label "MD_UP"
 		(at 72.39 77.47 0)
-		(fields_autoplaced yes)
 		(effects
 			(font
@@
 	(label "MD_DOWN"
 		(at 248.92 36.83 0)
-		(fields_autoplaced yes)
 		(effects
 			(font
@@
 	(label "C64_C"
 		(at 128.27 85.09 180)
-		(fields_autoplaced yes)
 		(effects
 			(font
@@
 	(label "C64_C"
 		(at 76.2 38.1 180)
-		(fields_autoplaced yes)
 		(effects
 			(font
@@
 	(label "MD_RIGHT_M"
 		(at 248.92 26.67 0)
-		(fields_autoplaced yes)
 		(effects
 			(font
@@
 	(label "MD_C"
 		(at 95.25 148.59 180)
-		(fields_autoplaced yes)
 		(effects
 			(font
@@
 	(label "C64_C"
 		(at 15.24 30.48 270)
-		(fields_autoplaced yes)
 		(effects
 			(font
@@
 	(label "MD_RIGHT"
 		(at 95.25 156.21 180)
-		(fields_autoplaced yes)
 		(effects
 			(font
@@
 	(label "MD_UP"
 		(at 20.32 72.39 0)
-		(fields_autoplaced yes)
 		(effects
 			(font
@@
 	(label "C64_UP"
 		(at 195.58 40.64 180)
-		(fields_autoplaced yes)
 		(effects
 			(font
@@
 	(label "MD_B{slash}~{A}"
 		(at 248.92 39.37 0)
-		(fields_autoplaced yes)
 		(effects
 			(font
@@
 	(label "MD_C"
 		(at 20.32 77.47 0)
-		(fields_autoplaced yes)
 		(effects
 			(font
@@
 	(label "CLK"
 		(at 260.35 132.08 0)
-		(fields_autoplaced yes)
 		(effects
 			(font
@@
 	(label "MD_A"
 		(at 72.39 95.25 0)
-		(fields_autoplaced yes)
 		(effects
 			(font
@@
 	(label "C64_POTY"
 		(at 177.8 20.32 180)
-		(fields_autoplaced yes)
 		(effects
 			(font
@@
 	(label "C64_FIRE"
 		(at 195.58 38.1 180)
-		(fields_autoplaced yes)
 		(effects
 			(font
@@
 	(label "MD_RIGHT"
 		(at 233.68 25.4 180)
-		(fields_autoplaced yes)
 		(effects
 			(font
@@
 	(label "MD_RIGHT_M"
 		(at 30.48 156.21 0)
-		(fields_autoplaced yes)
 		(effects
 			(font
@@
 	(label "MD_LEFT"
 		(at 233.68 30.48 180)
-		(fields_autoplaced yes)
 		(effects
 			(font
@@
 	(label "MD_UP"
 		(at 233.68 40.64 180)
-		(fields_autoplaced yes)
 		(effects
 			(font
@@
 	(label "C64_POTX"
 		(at 87.63 63.5 90)
-		(fields_autoplaced yes)
 		(effects
 			(font
@@
 	(label "MD_B{slash}~{A}"
 		(at 115.57 151.13 0)
-		(fields_autoplaced yes)
 		(effects
 			(font
@@
 	(label "MD_LEFT_M"
 		(at 30.48 153.67 0)
-		(fields_autoplaced yes)
 		(effects
 			(font
@@
 	(label "C64_POTX"
 		(at 177.8 22.86 180)
-		(fields_autoplaced yes)
 		(effects
 			(font
@@
 	(label "C64_LEFT"
 		(at 195.58 30.48 180)
-		(fields_autoplaced yes)
 		(effects
 			(font
@@
 			)
 		)
-		(property "Value" "10uF"
+		(property "Value" "10nF"
 			(at 207.01 140.9636 0)
 			(effects
@@
 			)
 		)
-		(property "Value" "47K"
+		(property "Value" "10K"
 			(at 271.78 144.78 90)
 			(effects

Commit message: Correct connection mistake
Connections:
- net C64_UP: no longer J2.1, RN1.5 (R4.2), U1.1, U3.2 (I0a)
- new net MD_UP: J2.1, RN1.5 (R4.2), U1.1, U3.2 (I0a)
Changed lines of the file:
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@@
-	(wire
-		(pts
-			(xy 185.42 40.64) (xy 233.68 40.64)
-		)
-		(stroke
-			(width 0)
-			(type default)
-		)
-	)
 	(wire
 		(pts
@@
 		(pts
 			(xy 163.83 22.86) (xy 177.8 22.86)
+		)
+		(stroke
+			(width 0)
+			(type default)
+		)
+	)
+	(wire
+		(pts
+			(xy 185.42 40.64) (xy 195.58 40.64)
 		)
 		(stroke
@@
 		(effects
 			(font
-				(size 1.27 1.27)
-			)
-			(justify right bottom)
-		)
-	)
-	(label "MD_UP"
-		(at 233.68 40.64 180)
-		(effects
-			(font
