File: MDC64Padapter.kicad_sch (KiCad schematic)
At the start: 44 parts, among them J1 DB9_F_TO_C64, J2 DB9_M_TO_PAD, Q1 BC847, Q2 BC847, SW1 MODE, U1 74ACT08, U2 74ACT373, U3 74ACT157, U4 74ACT373, U5 74AHC1G04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

Commit message: Update wrong LCSC numbers for two capacitors
Parts:
- C1, C2: LCSC PN C60133 -> C83170
Changed lines of the file:
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@@
 			)
 		)
-		(property "LCSC PN" "C60133"
+		(property "LCSC PN" "C83170"
 			(at 209.55 139.7 0)
 			(effects
@@
 			)
 		)
-		(property "LCSC PN" "C60133"
+		(property "LCSC PN" "C83170"
 			(at 227.33 137.16 90)
 			(effects

Commit message: Fixed a part number and add fabrication files for PCBWay and JLCPCB
Parts:
- U5: LCSC PN C19829641 -> C148197
Changed lines of the file:
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@@
 			)
 		)
-		(property "LCSC PN" "C19829641"
+		(property "LCSC PN" "C148197"
 			(at 227.33 109.22 0)
 			(effects
